File: PCB/Flight Controller.brd (EAGLE design)
At the start: 34.3 x 47.9 mm, 29 parts, among them J1 ZX62-AB-5PA(31), J2 M50-3600542R, U1 BMP390L, U2 NINA-B306, U4 BNO055, U5 LMS8117AMP-3.3/NOPB

Commit message: updated silkscreen and processed CAM job
Routing:
- net GND: track 96.1 -> 98.0 mm
Other:
- board text added: "Board Design by Josh Stidham"
- board text added: "Quadcopter Flight Controller V1"
